File: Raspberry_Pico_Breakout.kicad_pcb (KiCad board)
At the start: 2 copper layers, 48 x 63.5 mm, 16 parts, among them J1 Conn_01x20, J2 Conn_01x20, J3 Conn_01x20, J4 Conn_01x20, J5 Conn_01x20, J6 Conn_01x20, J7 Conn_01x20, J8 Conn_01x20

Commit message: doc: updated on schematic and PCB added license and design text
Other:
- board text added: "Licensed under CERN-OHL-W v2.0"
- board text added: "Mechaxil Approved Design"
Changed lines of the file:
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@@
+		)
+	)
+	(gr_text "Licensed under CERN-OHL-W v2.0"
+		(at 154.15 126.3 0)
+		(layer "B.SilkS")
+		(effects
+			(font
+				(size 1 1)
+				(thickness 0.1)
+			)
+			(justify bottom mirror)
 		)
 	)
@@
 		)
 	)
+	(gr_text "Mechaxil Approved Design"
+		(at 153.65 124.3 0)
+		(layer "B.SilkS")
+		(effects
+			(font
+				(size 1 1)
+				(thickness 0.1)
+			)
+			(justify bottom mirror)
+		)
+	)

Commit message: major: upgrade to KiCAD 10.0 and OSHW License
Parts:
- added G***: LOGO, assets:OSHW_Mark, B.Cu at (153.2, 126.3)
- G***: footprint Mechaxil Misc:Logo -> assets:Logo
