File: Raspberry_Pico_Breakout.kicad_pcb (KiCad board)
At the start: 2 copper layers, 48 x 63.5 mm, 17 parts, among them J1 Conn_01x20, J2 Conn_01x20, J3 Conn_01x20, J4 Conn_01x20, J5 Conn_01x20, J6 Conn_01x20, J7 Conn_01x20, J8 Conn_01x20

Commit message: feat: Probe GND pad for easy oscilloscope attachment
Parts:
- removed kibuzzard-69C7C267: G***, kibuzzard-69C7C267
- added TP1: TestPoint_Probe, TestPoint:TestPoint_Loop_D2.50mm_Drill1.0mm_LowProfile, F.Cu at (153.5, 124.6)
- added kibuzzard-6A0C12EA: G***, kibuzzard-6A0C12EA, F.Cu at (153.3, 76.2)
- added kibuzzard-6A0C1342: G***, kibuzzard-6A0C1342, F.Cu at (153.4, 121.1)
- moved G*** 56.0 mm to (152.9, 70.3)
Connections:
- net /GND renamed GND
Routing:
- net GND: track 0.00 -> 53.3 mm
- net /GPIO21: track 7.62 -> 15.3 mm
- net /GPIO2: track 7.63 -> 15.3 mm
- net /GPIO15: track 7.63 -> 15.3 mm
- net /GPIO9: track 7.63 -> 15.3 mm
- net /GPIO8: track 7.63 -> 15.3 mm
- net /GPIO7: track 7.63 -> 15.3 mm
- net /GPIO6: track 7.63 -> 15.3 mm
- net /GPIO5: track 7.63 -> 15.3 mm
- net /GPIO4: track 7.63 -> 15.3 mm
- net /GPIO3: track 7.63 -> 15.3 mm
- net /GPIO14: track 7.63 -> 15.3 mm
- net /GPIO13: track 7.63 -> 15.3 mm
- net /GPIO12: track 7.63 -> 15.3 mm
- net /GPIO11: track 7.63 -> 15.3 mm
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